Commit message: tiago: fix self collisions, add single arm tiago

File: gibson2/assets/models/tiago/tiago_dual.urdf (robot description, URDF)
Before this commit: robot tiago_dual, 104 links, 103 joints
Links:
- removed link base_mic_back_left_link
- removed link base_mic_back_right_link
- removed link base_mic_front_left_link
- removed link base_mic_front_right_link
- removed link caster_back_left_1_link
- removed link caster_back_left_2_link
- removed link caster_back_right_1_link
- removed link caster_back_right_2_link
- removed link caster_front_left_1_link
- removed link caster_front_left_2_link
- removed link caster_front_right_1_link
- removed link caster_front_right_2_link
- removed link hand_right_grasping_frame
- removed link hand_right_index_abd_link
- removed link hand_right_index_flex_1_link
- removed link hand_right_index_flex_2_link
- removed link hand_right_index_flex_3_link
- removed link hand_right_index_link
- removed link hand_right_index_virtual_1_link
- removed link hand_right_index_virtual_2_link
- removed link hand_right_index_virtual_3_link
- removed link hand_right_little_abd_link
- removed link hand_right_little_flex_1_link
- removed link hand_right_little_flex_2_link
- removed link hand_right_little_flex_3_link
- removed link hand_right_little_virtual_1_link
- removed link hand_right_little_virtual_2_link
- removed link hand_right_little_virtual_3_link
- removed link hand_right_middle_abd_link
- removed link hand_right_middle_flex_1_link
- removed link hand_right_middle_flex_2_link
- removed link hand_right_middle_flex_3_link
- removed link hand_right_middle_virtual_1_link
- removed link hand_right_middle_virtual_2_link
- removed link hand_right_middle_virtual_3_link
- removed link hand_right_mrl_link
- removed link hand_right_palm_link
- removed link hand_right_ring_abd_link
- removed link hand_right_ring_flex_1_link
- removed link hand_right_ring_flex_2_link
- removed link hand_right_ring_flex_3_link
- removed link hand_right_ring_virtual_1_link
- removed link hand_right_ring_virtual_2_link
- removed link hand_right_ring_virtual_3_link
- removed link hand_right_safety_box
- removed link hand_right_thumb_abd_link
- removed link hand_right_thumb_flex_1_link
- removed link hand_right_thumb_flex_2_link
- removed link hand_right_thumb_link
- removed link hand_right_thumb_virtual_1_link
- removed link hand_right_thumb_virtual_2_link
- removed link hand_right_tool_link
- removed link suspension_left_link
- removed link suspension_right_link
- added link ignore_caster_back_left_1_link, mass 0.05144761; visual mesh filename=package://pmb2_description/meshes/wheels/caster_1.stl
- added link ignore_caster_back_left_2_link, mass 0.08855784; collision cylinder length=0.015 radius=0.025; visual mesh filename=package://pmb2_description/meshes/wheels/caster_2.stl
- added link ignore_caster_back_right_1_link, mass 0.05144761; visual mesh filename=package://pmb2_description/meshes/wheels/caster_1.stl
- added link ignore_caster_back_right_2_link, mass 0.08855784; collision cylinder length=0.015 radius=0.025; visual mesh filename=package://pmb2_description/meshes/wheels/caster_2.stl
- added link ignore_caster_front_left_1_link, mass 0.05144761; visual mesh filename=package://pmb2_description/meshes/wheels/caster_1.stl
- added link ignore_caster_front_left_2_link, mass 0.08855784; collision cylinder length=0.015 radius=0.025; visual mesh filename=package://pmb2_description/meshes/wheels/caster_2.stl
- added link ignore_caster_front_right_1_link, mass 0.05144761; visual mesh filename=package://pmb2_description/meshes/wheels/caster_1.stl
- added link ignore_caster_front_right_2_link, mass 0.08855784; collision cylinder length=0.015 radius=0.025; visual mesh filename=package://pmb2_description/meshes/wheels/caster_2.stl
- added link ignore_suspension_left_link, mass 10
- added link ignore_suspension_right_link, mass 10
- link base_footprint: mass None -> 0.001
Joints:
- removed joint base_mic_back_left_joint
- removed joint base_mic_back_right_joint
- removed joint base_mic_front_left_joint
- removed joint base_mic_front_right_joint
- removed joint caster_back_left_1_joint
- removed joint caster_back_left_2_joint
- removed joint caster_back_right_1_joint
- removed joint caster_back_right_2_joint
- removed joint caster_front_left_1_joint
- removed joint caster_front_left_2_joint
- removed joint caster_front_right_1_joint
- removed joint caster_front_right_2_joint
- removed joint hand_right_grasping_fixed_joint
- removed joint hand_right_index_abd_joint
- removed joint hand_right_index_flex_1_joint
- removed joint hand_right_index_flex_2_joint
- removed joint hand_right_index_flex_3_joint
- removed joint hand_right_index_joint
- removed joint hand_right_index_virtual_1_joint
- removed joint hand_right_index_virtual_2_joint
- removed joint hand_right_index_virtual_3_joint
- removed joint hand_right_little_abd_joint
- removed joint hand_right_little_flex_1_joint
- removed joint hand_right_little_flex_2_joint
- removed joint hand_right_little_flex_3_joint
- removed joint hand_right_little_virtual_1_joint
- removed joint hand_right_little_virtual_2_joint
- removed joint hand_right_little_virtual_3_joint
- removed joint hand_right_middle_abd_joint
- removed joint hand_right_middle_flex_1_joint
- removed joint hand_right_middle_flex_2_joint
- removed joint hand_right_middle_flex_3_joint
- removed joint hand_right_middle_virtual_1_joint
- removed joint hand_right_middle_virtual_2_joint
- removed joint hand_right_middle_virtual_3_joint
- removed joint hand_right_mrl_joint
- removed joint hand_right_palm_joint
- removed joint hand_right_ring_abd_joint
- removed joint hand_right_ring_flex_1_joint
- removed joint hand_right_ring_flex_2_joint
- removed joint hand_right_ring_flex_3_joint
- removed joint hand_right_ring_virtual_1_joint
- removed joint hand_right_ring_virtual_2_joint
- removed joint hand_right_ring_virtual_3_joint
- removed joint hand_right_safety_box_joint
- removed joint hand_right_thumb_abd_joint
- removed joint hand_right_thumb_flex_1_joint
- removed joint hand_right_thumb_flex_2_joint
- removed joint hand_right_thumb_joint
- removed joint hand_right_thumb_virtual_1_joint
- removed joint hand_right_thumb_virtual_2_joint
- removed joint hand_right_tool_joint
- removed joint suspension_left_joint
- removed joint suspension_right_joint
- added joint ignore_caster_back_left_1_joint: type continuous, parent base_link, child ignore_caster_back_left_1_link, origin xyz=-0.1735 0.102 -0.0335 rpy=0 0 0, axis 0 0 1
- added joint ignore_caster_back_left_2_joint: type continuous, parent ignore_caster_back_left_1_link, child ignore_caster_back_left_2_link, origin xyz=-0.016 0.0000 -0.040 rpy=-1.57079632679 0 0, axis 0 0 1
- added joint ignore_caster_back_right_1_joint: type continuous, parent base_link, child ignore_caster_back_right_1_link, origin xyz=-0.1735 -0.102 -0.0335 rpy=0 0 0, axis 0 0 1
- added joint ignore_caster_back_right_2_joint: type continuous, parent ignore_caster_back_right_1_link, child ignore_caster_back_right_2_link, origin xyz=-0.016 0.0000 -0.040 rpy=-1.57079632679 0 0, axis 0 0 1
- added joint ignore_caster_front_left_1_joint: type continuous, parent base_link, child ignore_caster_front_left_1_link, origin xyz=0.1695 0.102 -0.0335 rpy=0 0 0, axis 0 0 1
- added joint ignore_caster_front_left_2_joint: type continuous, parent ignore_caster_front_left_1_link, child ignore_caster_front_left_2_link, origin xyz=-0.016 0.0000 -0.040 rpy=-1.57079632679 0 0, axis 0 0 1
- added joint ignore_caster_front_right_1_joint: type continuous, parent base_link, child ignore_caster_front_right_1_link, origin xyz=0.1695 -0.102 -0.0335 rpy=0 0 0, axis 0 0 1
- added joint ignore_caster_front_right_2_joint: type continuous, parent ignore_caster_front_right_1_link, child ignore_caster_front_right_2_link, origin xyz=-0.016 0.0000 -0.040 rpy=-1.57079632679 0 0, axis 0 0 1
- added joint ignore_suspension_left_joint: type prismatic, parent base_link, child ignore_suspension_left_link, origin xyz=0 0 0 rpy=0 0 0, axis 0 0 1, limit lower=-0.005 upper=0.005 effort=100.0 velocity=1.0
- added joint ignore_suspension_right_joint: type prismatic, parent base_link, child ignore_suspension_right_link, origin xyz=0 0 0 rpy=0 0 0, axis 0 0 1, limit lower=-0.005 upper=0.005 effort=100.0 velocity=1.0
- joint wheel_left_joint: parent suspension_left_link -> ignore_suspension_left_link
- joint wheel_right_joint: parent suspension_right_link -> ignore_suspension_right_link
