Commit message: add grasp detection and grasp simulation

File: gibson2/assets/models/tiago/tiago_dual_nohand.urdf (robot description, URDF)
Before this commit: robot tiago_dual, 99 links, 98 joints
Links:
- removed link hand_right_grasping_frame
- removed link hand_right_index_abd_link
- removed link hand_right_index_flex_1_link
- removed link hand_right_index_flex_2_link
- removed link hand_right_index_flex_3_link
- removed link hand_right_index_link
- removed link hand_right_index_virtual_1_link
- removed link hand_right_index_virtual_2_link
- removed link hand_right_index_virtual_3_link
- removed link hand_right_little_abd_link
- removed link hand_right_little_flex_1_link
- removed link hand_right_little_flex_2_link
- removed link hand_right_little_flex_3_link
- removed link hand_right_little_virtual_1_link
- removed link hand_right_little_virtual_2_link
- removed link hand_right_little_virtual_3_link
- removed link hand_right_middle_abd_link
- removed link hand_right_middle_flex_1_link
- removed link hand_right_middle_flex_2_link
- removed link hand_right_middle_flex_3_link
- removed link hand_right_middle_virtual_1_link
- removed link hand_right_middle_virtual_2_link
- removed link hand_right_middle_virtual_3_link
- removed link hand_right_mrl_link
- removed link hand_right_palm_link
- removed link hand_right_ring_abd_link
- removed link hand_right_ring_flex_1_link
- removed link hand_right_ring_flex_2_link
- removed link hand_right_ring_flex_3_link
- removed link hand_right_ring_virtual_1_link
- removed link hand_right_ring_virtual_2_link
- removed link hand_right_ring_virtual_3_link
- removed link hand_right_thumb_abd_link
- removed link hand_right_thumb_flex_1_link
- removed link hand_right_thumb_flex_2_link
- removed link hand_right_thumb_link
- removed link hand_right_thumb_virtual_1_link
- removed link hand_right_thumb_virtual_2_link
- removed link hand_right_tool_link
Joints:
- removed joint hand_right_grasping_fixed_joint
- removed joint hand_right_index_abd_joint
- removed joint hand_right_index_flex_1_joint
- removed joint hand_right_index_flex_2_joint
- removed joint hand_right_index_flex_3_joint
- removed joint hand_right_index_joint
- removed joint hand_right_index_virtual_1_joint
- removed joint hand_right_index_virtual_2_joint
- removed joint hand_right_index_virtual_3_joint
- removed joint hand_right_little_abd_joint
- removed joint hand_right_little_flex_1_joint
- removed joint hand_right_little_flex_2_joint
- removed joint hand_right_little_flex_3_joint
- removed joint hand_right_little_virtual_1_joint
- removed joint hand_right_little_virtual_2_joint
- removed joint hand_right_little_virtual_3_joint
- removed joint hand_right_middle_abd_joint
- removed joint hand_right_middle_flex_1_joint
- removed joint hand_right_middle_flex_2_joint
- removed joint hand_right_middle_flex_3_joint
- removed joint hand_right_middle_virtual_1_joint
- removed joint hand_right_middle_virtual_2_joint
- removed joint hand_right_middle_virtual_3_joint
- removed joint hand_right_mrl_joint
- removed joint hand_right_palm_joint
- removed joint hand_right_ring_abd_joint
- removed joint hand_right_ring_flex_1_joint
- removed joint hand_right_ring_flex_2_joint
- removed joint hand_right_ring_flex_3_joint
- removed joint hand_right_ring_virtual_1_joint
- removed joint hand_right_ring_virtual_2_joint
- removed joint hand_right_ring_virtual_3_joint
- removed joint hand_right_thumb_abd_joint
- removed joint hand_right_thumb_flex_1_joint
- removed joint hand_right_thumb_flex_2_joint
- removed joint hand_right_thumb_joint
- removed joint hand_right_thumb_virtual_1_joint
- removed joint hand_right_thumb_virtual_2_joint
- removed joint hand_right_tool_joint
